File: electrical/test_bench/TestBench.kicad_sch (KiCad schematic)
At the start: 27 parts, among them J1 DB9_Female, J2 DB9_Female, J3 Screw_Terminal, U1 MD10C-R3, U2 MD10C-R3, U3 LM7805_TO220, U4 ESP32-DEVKITC-32UE, U5 BOB-12009, U6 BOB-12009, U7 ACS711EX-15A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

Commit message: updated schematic title and added pdf
Other:
- company: (none) -> ENPH 459 Project Lab - Project 2402
- title: (none) -> ENPH 459 Dual Twiddlerino Test Bench Schematic
Changed lines of the file:
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@@
 (kicad_sch (version 20211123) (generator eeschema)
   (paper "A4")
+  (title_block
+    (title "ENPH 459 Dual Twiddlerino Test Bench Schematic")
+    (date "2024-04-08")
+    (rev "1.1")
+    (company "ENPH 459 Project Lab - Project 2402")
+  )
   (junction (at 45.72 44.45) (diameter 0) (color 0 0 0 0)
   )
